File: LEDClockControl/LEDClockControl.sch (KiCad schematic (older format))
At the start: 20 parts, among them J1 Barrel_Jack_Switch, J2 Conn_02x06_Odd_Even, J3 Conn_01x05, Q1 DMG2301L, Q2 DMG2301L, Q3 DMG2301L, Q4 DMG2301L, Q5 DMG2301L, Q6 DMG2301L, Q7 DMG2301L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

Commit message: Added RTC to schematic
Parts:
- added C5, C6: 12pF, Capacitor_SMD:C_0805_2012Metric_Pad1.15x1.40mm_HandSolder, symbol Device:C
- added R2, R3: 3k3, Resistor_SMD:R_0805_2012Metric_Pad1.15x1.40mm_HandSolder, symbol Device:R
- added U4: PCF8563T, Package_SO:SOP-8_6.62x9.15mm_P2.54mm, symbol Timer_RTC:PCF8563T
- added Y2: 32.768kHz, Crystal:Crystal_C26-LF_D2.1mm_L6.5mm_Horizontal, symbol Device:Crystal
- C1, C2: value 20pF -> 12pF; footprint Capacitor_SMD:C_1206_3216Metric_Pad1.42x1.75mm_HandSolder -> Capacitor_SMD:C_0805_2012Metric_Pad1.15x1.40mm_HandSolder; LCSC Number C1886 -> C152848
Connections:
- wire segments 112 -> 132
Other:
- moved on the sheet: U3
